Commit message: update

File: install/my_box_bot_gazebo/share/my_box_bot_gazebo/urdf/Assem1_urdf.urdf (robot description, URDF)
Before this commit: robot Assem1_urdf, 9 links, 8 joints
Links:
- added link world_link
- link acc1: geometry collision mesh filename=package:///meshes/acc1.STL; visual mesh filename=package:///meshes/acc1.STL
- link acc2: geometry collision mesh filename=package:///meshes/acc2.STL; visual mesh filename=package:///meshes/acc2.STL
- link base_link: geometry collision mesh filename=package:///meshes/base_link.STL; visual mesh filename=package:///meshes/base_link.STL
- link cbracket: geometry collision mesh filename=package:///meshes/cbracket.STL; visual mesh filename=package:///meshes/cbracket.STL
- link leg1: geometry collision mesh filename=package:///meshes/leg1.STL; visual mesh filename=package:///meshes/leg1.STL
- link leg2: geometry collision mesh filename=package:///meshes/leg2.STL; visual mesh filename=package:///meshes/leg2.STL
- link lowleg1: geometry collision mesh filename=package:///meshes/lowleg1.STL; visual mesh filename=package:///meshes/lowleg1.STL
- link lowleg2: geometry collision mesh filename=package:///meshes/lowleg2.STL; visual mesh filename=package:///meshes/lowleg2.STL
- link pulley: geometry collision mesh filename=package:///meshes/pulley.STL; visual mesh filename=package:///meshes/pulley.STL
Joints:
- added joint dummy_joint: type fixed, parent world_link, child base_link
- joint j4: limit lower=3.142 upper=-3.142 effort=200 velocity=3 -> lower=-3.142 upper=3.142 effort=200 velocity=3
- joint j5: limit lower=3.142 upper=-3.142 effort=200 velocity=3 -> lower=-3.142 upper=3.142 effort=200 velocity=3
