Commit message: update to urdf

File: install/my_box_bot_gazebo/share/my_box_bot_gazebo/urdf/final10_urdf.urdf (robot description, URDF)
Before this commit: robot titanleg, 5 links, 4 joints
Joints:
- joint cb_joint: axis 0 0 0 -> 0 -1 0; origin xyz=0.31938 -0.55114 0.47454 rpy=-1.5708 0 -1.5708 -> xyz=0.21565 -0.53088 0.5435 rpy=0 0 3.1416
- joint lower_joint: axis 0 0 0 -> -1 0 0; origin xyz=0.3406 -0.32494 -0.080516 rpy=0 0 1.527 -> xyz=-0.012 -0.0043465 -0.26991 rpy=0 0 0
- joint motor_leg_joint: axis 0 0 0 -> 1 0 0; origin xyz=-0.011894 0.010745 -0.16143 rpy=3.1416 0 0.010453 -> xyz=0.21211 0.089 0 rpy=0 0 0
