Commit message: position movement updated

File: install/my_box_bot_gazebo/share/my_box_bot_gazebo/urdf/final12_urdf.urdf (robot description, URDF)
Before this commit: robot titanleg, 5 links, 4 joints
Joints:
- joint lower_joint: limit lower=0 upper=0 effort=0 velocity=0 -> lower=0 upper=3.14 effort=1.0 velocity=1.0

File: src/my_box_bot_gazebo/urdf/final12_urdf.urdf (robot description, URDF)
Before this commit: robot titanleg, 5 links, 4 joints
Joints:
- joint lower_joint: limit lower=0 upper=0 effort=0 velocity=0 -> lower=0 upper=3.14 effort=1.0 velocity=1.0

Commit message: update

File: install/my_box_bot_gazebo/share/my_box_bot_gazebo/urdf/final12_urdf.urdf (robot description, URDF)
Before this commit: robot titanleg, 5 links, 4 joints
Joints:
- joint cb_joint: limit lower=0 upper=0 effort=0 velocity=0 -> lower=0 upper=6.28 effort=1.0 velocity=1.0
- joint motor_leg_joint: limit lower=0 upper=0 effort=0 velocity=0 -> lower=0 upper=6.28 effort=1.0 velocity=1.0

File: src/my_box_bot_gazebo/urdf/final12_urdf.urdf (robot description, URDF)
Before this commit: robot titanleg, 5 links, 4 joints
Joints:
- joint cb_joint: limit lower=0 upper=0 effort=0 velocity=0 -> lower=0 upper=6.28 effort=1.0 velocity=1.0
- joint motor_leg_joint: limit lower=0 upper=0 effort=0 velocity=0 -> lower=0 upper=6.28 effort=1.0 velocity=1.0
