Commit message: updates

File: src/my_box_bot_gazebo/urdf/final2_urdf.urdf (robot description, URDF)
Before this commit: robot titanleg, 8 links, 7 joints
Links:
- removed link acc
- removed link acc_knee
- removed link upperleg
- added link abd_acc, mass 0.580805573486017; collision mesh filename=package://my_box_bot_gazebo/meshes/abd_acc.STL; visual mesh filename=package://my_box_bot_gazebo/meshes/abd_acc.STL
- added link knee_acc, mass 0.487854303371581; collision mesh filename=package://my_box_bot_gazebo/meshes/knee_acc.STL; visual mesh filename=package://my_box_bot_gazebo/meshes/knee_acc.STL
- added link upperleg1, mass 0.365894283988061; collision mesh filename=package://my_box_bot_gazebo/meshes/upperleg1.STL; visual mesh filename=package://my_box_bot_gazebo/meshes/upperleg1.STL
- added link upperleg2, mass 0.365892540566899; collision mesh filename=package://my_box_bot_gazebo/meshes/upperleg2.STL; visual mesh filename=package://my_box_bot_gazebo/meshes/upperleg2.STL
- link base_link: mass 3.0381 -> 4.56027988555656
- link c_bracket: mass 0.19414 -> 0.1941398277098
- link lowerleg: mass 0.66281 -> 0.66280770717818
- link pulley: mass 0.15149 -> 0.15148726652934
Joints:
- removed joint acc_abd_knee
- removed joint acc_pulley
- removed joint acc_ul
- removed joint adb_knee
- removed joint pulley_lowl
- added joint knee_joint: type revolute, parent abd_acc, child knee_acc, origin xyz=-0.0281 0.015201 0.109 rpy=0 0 -0.53405, axis 0 0 0, limit lower=0 upper=0 effort=0 velocity=0
- added joint leg1: type fixed, parent knee_acc, child upperleg1, origin xyz=0.013735 0.058961 0.18616 rpy=3.1416 0 2.0944, axis 0 0 0
- added joint leg_joint2: type fixed, parent knee_acc, child upperleg2, origin xyz=0.013735 0.058961 0.21416 rpy=0 0 -1.0472, axis 0 0 0
- added joint lowerleg_joint: type revolute, parent pulley, child lowerleg, origin xyz=0.38429 0.29106 0.22292 rpy=-3.1416 0 -1.8781, axis 0 0 0, limit lower=0 upper=0 effort=0 velocity=0
- added joint pulley_joint: type revolute, parent knee_acc, child pulley, origin xyz=0.013735 0.058961 0.21416 rpy=3.1416 0 -1.3981, axis 0 0 0, limit lower=0 upper=0 effort=0 velocity=0
- added joint shoulder_joint: type fixed, parent c_bracket, child abd_acc, origin xyz=0.058961 0.013735 0.086158 rpy=3.1416 0 -1.5708, axis 0 0 0
